Commit message: Set the slave finger torque limit to the EL05 output torque (1.1 Nm)
The released slave uses the RobStride EL05 finger motor, limited in
hardware to 1.1 Nm for continuous stall. Define the effort once in the
Xacro macro; the MJCF actuator forcerange is now generated from the URDF
effort instead of a hard-coded 4 Nm, and the USD drive maxForce follows.
Record the motor in model.json, update the slave READMEs, and test that
URDF, MJCF and USD agree on the limit.

Co-Authored-By: Claude Opus 5.5 <noreply@anthropic.com>

File: ros/taccap_description/urdf/taccap_g1_slave.urdf (robot description, URDF)
Before this commit: robot taccap_g1_slave, 6 links, 5 joints
Joints:
- joint taccap_left_finger_joint: limit lower=-0.5047492196767601 upper=0 effort=4 velocity=1 -> lower=-0.5047492196767601 upper=0 effort=1.1 velocity=1
- joint taccap_right_finger_joint: limit lower=0 upper=0.5047492196767601 effort=4 velocity=1 -> lower=0 upper=0.5047492196767601 effort=1.1 velocity=1

File: ros/taccap_description/urdf/taccap_g1_slave_macro.xacro (robot description, xacro)
@@ -2,4 +2,7 @@
 <robot xmlns:xacro="http://www.ros.org/wiki/xacro">
   <!-- Mechanical description of the TacCap G1 slave gripper. -->
+  <!-- Maximum output torque (N m) of the finger motor, RobStride EL05; the hardware limits it to
+       1.1 N m for continuous stall. MJCF and USD take their force limits from this effort. -->
+  <xacro:property name="taccap_finger_effort" value="1.1"/>
   <xacro:macro name="taccap_g1_slave" params="prefix:='' with_mount:=false mesh_root:='package://taccap_description/meshes'">
     <material name="${prefix}taccap_base_mat"><color rgba="0.75294 0.75294 0.75294 1"/></material>
@@ -64,6 +67,6 @@
       <origin xyz="0.0120336718 0.0199500106 0.0484999712" rpy="0 0 0"/>
       <axis xyz="1 0 0"/>
-      <!-- Effort and velocity are simulation settings; see config/model.json. -->
-      <limit lower="-0.5047492196767601" upper="0" effort="4" velocity="1"/>
+      <!-- Effort is the finger motor's maximum output torque; see config/model.json. -->
+      <limit lower="-0.5047492196767601" upper="0" effort="${taccap_finger_effort}" velocity="1"/>
       <dynamics damping="0.08" friction="0.01"/>
       <mimic joint="${prefix}taccap_right_finger_joint" multiplier="-1" offset="0"/>
@@ -85,5 +88,5 @@
       <origin xyz="0.0120336718 -0.0199499894 0.0484999712" rpy="0 0 0"/>
       <axis xyz="1 0 0"/>
-      <limit lower="0" upper="0.5047492196767601" effort="4" velocity="1"/>
+      <limit lower="0" upper="0.5047492196767601" effort="${taccap_finger_effort}" velocity="1"/>
       <dynamics damping="0.08" friction="0.01"/>
     </joint>

File: ros/taccap_description/urdf/taccap_g1_slave_with_mount.urdf (robot description, URDF)
Before this commit: robot taccap_g1_slave_with_mount, 7 links, 6 joints
Joints:
- joint taccap_left_finger_joint: limit lower=-0.5047492196767601 upper=0 effort=4 velocity=1 -> lower=-0.5047492196767601 upper=0 effort=1.1 velocity=1
- joint taccap_right_finger_joint: limit lower=0 upper=0.5047492196767601 effort=4 velocity=1 -> lower=0 upper=0.5047492196767601 effort=1.1 velocity=1
