Commit message: feat: update slave physics and models to v2026.10.23
Use the locked upstream URDF geometry, masses, COMs, full inertia tensors
and finger measurement-pose corrections. Retain downstream root interfaces
and the confirmed 1.1 Nm EL05 effort. Bare/mounted masses are 0.750/0.785 kg.
Generate matching MJCF/USD, include simplified collision resources in the
wheel, and filter internal motor/finger convex-hull overlap in simulation.

Record exhaustive three-way XML/file differences and independently
recompute six parts' physics from the upstream SW inputs. Verify commit
attribution against every source file before allowing a future revision pin.

Validation: 107 tests passed; import/slave/master generators --check;
live source hash audit; wheel/sdist build and independent wheel installation.
No ROS/Isaac Sim/hardware runtime validation performed.

Upstream-Repository: https://github.com/XenseRobotics-AI/xense-description.git
Upstream-Path: assets/grippers/xense/taccap/slave-v2026.10.23
Upstream-Lock: vendor/taccap_slave/upstream.json
Upstream-Revision: pending (uncommitted worktree snapshot)

File: ros/taccap_description/urdf/taccap_g1_slave.urdf (robot description, URDF)
Before this commit: robot taccap_g1_slave, 6 links, 5 joints
Links:
- added link taccap_camera_body_link, mass 0.018; collision mesh filename=../meshes/camera_link.STL; visual mesh filename=../meshes/camera_link.STL
- added link taccap_motor_link, mass 0.299; collision mesh filename=../meshes/collision/motor_link.stl; visual mesh filename=../meshes/motor_link.STL
- link taccap_base_link: mass 0.415 -> 0.153; geometry collision mesh filename=../meshes/collision/body_link.stl; visual mesh filename=../meshes/body_link.STL
- link taccap_left_finger_link: mass 0.36678 -> 0.14; geometry collision mesh filename=../meshes/collision/left_link.stl; visual mesh filename=../meshes/left_link.STL
- link taccap_right_finger_link: mass 0.36678 -> 0.14; geometry collision mesh filename=../meshes/collision/right_link.stl; visual mesh filename=../meshes/right_link.STL
Joints:
- added joint taccap_camera_body_joint: type fixed, parent taccap_base_link, child taccap_camera_body_link, origin xyz=0 0 0 rpy=0 0 0
- added joint taccap_motor_joint: type fixed, parent taccap_base_link, child taccap_motor_link, origin xyz=0 0 0 rpy=0 0 0

File: ros/taccap_description/urdf/taccap_g1_slave_macro.xacro (robot description, xacro)
@@ -1,115 +1,190 @@
-<?xml version="1.0"?>
 <robot xmlns:xacro="http://www.ros.org/wiki/xacro">
-  <!-- Mechanical description of the TacCap G1 slave gripper. -->
-  <!-- Maximum output torque (N m) of the finger motor, RobStride EL05; the hardware limits it to
-       1.1 N m for continuous stall. MJCF and USD take their force limits from this effort. -->
-  <xacro:property name="taccap_finger_effort" value="1.1"/>
+  <!-- Generated by scripts/import_slave.py from the locked upstream snapshot. -->
   <xacro:macro name="taccap_g1_slave" params="prefix:='' with_mount:=false mesh_root:='package://taccap_description/meshes'">
-    <material name="${prefix}taccap_base_mat"><color rgba="0.75294 0.75294 0.75294 1"/></material>
-    <material name="${prefix}taccap_left_mat"><color rgba="1 1 1 1"/></material>
-    <material name="${prefix}taccap_right_mat"><color rgba="0.60392 0.60392 0.60392 1"/></material>
-    <material name="${prefix}taccap_mount_mat"><color rgba="0.89804 0.91765 0.92941 1"/></material>
-    <!-- taccap_base_link: gripper mounting face (body/Asm_link mating face). +Z along the tool
-         axis, +Y toward the left finger, +X toward the off-axis fingers. Meshes keep their native
-         CAD frame (+X tool axis); their placement is the origin below. -->
-    <xacro:property name="cad_xyz" value="0.01975 -0.0060769 0.034023"/>
-    <xacro:property name="cad_rpy" value="0 ${-pi/2} 0"/>
-    <xacro:if value="${with_mount}">
-      <!-- Optional adapter; its robot-side face is the root and attaches to the arm flange. -->
-      <link name="${prefix}taccap_mount_link">
-        <visual name="${prefix}asm_visual">
-          <origin xyz="0 0 0" rpy="${cad_rpy}"/>
-          <geometry><mesh filename="${mesh_root}/Asm_link.STL"/></geometry>
-          <material name="${prefix}taccap_mount_mat"/>
-        </visual>
-        <collision name="${prefix}asm_collision">
-          <origin xyz="0 0 0" rpy="${cad_rpy}"/>
-          <geometry><mesh filename="${mesh_root}/Asm_link.STL"/></geometry>
-        </collision>
-      </link>
-      <joint name="${prefix}taccap_mount_joint" type="fixed">
-        <parent link="${prefix}taccap_mount_link"/><child link="${prefix}taccap_base_link"/>
-        <origin xyz="0 0 0.012" rpy="0 0 0"/>
-      </joint>
-    </xacro:if>
+    <material name="${prefix}taccap_base_mat">
+      <color rgba="0.75294 0.75294 0.75294 1" />
+    </material>
+    <material name="${prefix}taccap_left_mat">
+      <color rgba="1 1 1 1" />
+    </material>
+    <material name="${prefix}taccap_right_mat">
+      <color rgba="0.60392 0.60392 0.60392 1" />
+    </material>
+    <material name="${prefix}taccap_cover_mat">
+      <color rgba="0.89804 0.91765 0.92941 1" />
+    </material>
     <link name="${prefix}taccap_base_link">
-      <!-- Body inertial in the base frame. -->
       <inertial>
-        <origin xyz="0.010155 -0.0007499 0.0361" rpy="0 0 0"/>
-        <mass value="0.415"/>
-        <inertia ixx="0.000573" iyy="0.000748" izz="0.000680" ixy="0" ixz="0" iyz="0"/>
+        <origin xyz="0.00055404 -0.0011065 0.03389788000000001" rpy="0 0 0" />
+        <mass value="0.153" />
+        <inertia ixx="0.0001662522337781271" ixy="5.051220230199417e-07" ixz="1.023875307549503e-05" iyy="0.000126891433023779" iyz="-1.820980122271716e-06" izz="0.0001290344694980937" />
       </inertial>
-      <visual name="${prefix}base_visual">
-        <origin xyz="${cad_xyz}" rpy="${cad_rpy}"/>
-        <geometry><mesh filename="${mesh_root}/base_link.STL"/></geometry><material name="${prefix}taccap_base_mat"/>
+      <visual name="${prefix}body_link_visual">
+        <origin xyz="0.01975 -0.0060769 0.034023" rpy="-0 -1.570796326794897 0" />
+        <geometry>
+          <mesh filename="${mesh_root}/body_link.STL" />
+        </geometry>
+        <material name="${prefix}taccap_base_mat" />
       </visual>
-      <collision name="${prefix}base_collision">
-        <origin xyz="${cad_xyz}" rpy="${cad_rpy}"/>
-        <geometry><mesh filename="${mesh_root}/base_link.STL"/></geometry>
+      <collision name="${prefix}body_link_collision">
+        <origin xyz="0.01975 -0.0060769 0.034023" rpy="-0 -1.570796326794897 0" />
+        <geometry>
+          <mesh filename="${mesh_root}/collision/body_link.stl" />
+        </geometry>
+      </collision>
+    </link>
+    <link name="${prefix}taccap_motor_link">
+      <inertial>
+        <origin xyz="0.03743085 -0.00109355 0.02554797" rpy="0 0 0" />
+        <mass value="0.299" />
+        <inertia ixx="2.530466922324684e-05" ixy="-2.027952739115101e-06" ixz="-1.239938363961379e-07" iyy="4.01613260249333e-05" iyz="-7.393526076882528e-07" izz="4.954026835181985e-05" />
+      </inertial>
+      <visual name="${prefix}motor_link_visual">
+        <origin xyz="0.01975 -0.0060769 0.034023" rpy="-0 -1.570796326794897 0" />
+        <geometry>
+          <mesh filename="${mesh_root}/motor_link.STL" />
+        </geometry>
+        <material name="${prefix}taccap_base_mat" />
+      </visual>
+      <collision name="${prefix}motor_link_collision">
+        <origin xyz="0.01975 -0.0060769 0.034023" rpy="-0 -1.570796326794897 0" />
+        <geometry>
+          <mesh filename="${mesh_root}/collision/motor_link.stl" />
+        </geometry>
       </collision>
     </link>
     <link name="${prefix}taccap_left_finger_link">
       <inertial>
-        <origin xyz="0.020693 -0.00669 0.074921" rpy="0 0 0"/>
-        <mass value="0.36678"/>
-        <inertia ixx="0.00015235" iyy="0.00015466" izz="3.3606e-05" ixy="2.9254e-07" ixz="-2.4362e-06" iyz="-6.6715e-06"/>
+        <origin xyz="0.0140949482 -0.00330133312635219 0.04838757908594267" rpy="0 0 0" />
+        <mass value="0.14" />
+        <inertia ixx="0.0003065325738824327" ixy="1.304843016703693e-06" ixz="-6.577075277330767e-05" iyy="0.0003222085257195986" iyz="7.713878953415112e-06" izz="3.792830299796826e-05" />
       </inertial>
-      <visual name="${prefix}left_finger_visual">
-        <origin xyz="0 0 0" rpy="${cad_rpy}"/>
-        <geometry><mesh filename="${mesh_root}/grip_left.STL"/></geometry><material name="${prefix}taccap_left_mat"/>
+      <visual name="${prefix}left_link_visual">
+        <origin xyz="1.776356839400251e-18 0 0" rpy="1.570796326794894 -1.513048197635941 -1.570796326794894" />
+        <geometry>
+          <mesh filename="${mesh_root}/left_link.STL" />
+        </geometry>
+        <material name="${prefix}taccap_left_mat" />
       </visual>
-      <collision name="${prefix}left_finger_collision"><origin xyz="0 0 0" rpy="${cad_rpy}"/><geometry><mesh filename="${mesh_root}/grip_left.STL"/></geometry></collision>
+      <collision name="${prefix}left_link_collision">
+        <origin xyz="1.776356839400251e-18 0 0" rpy="1.570796326794894 -1.513048197635941 -1.570796326794894" />
+        <geometry>
+          <mesh filename="${mesh_root}/collision/left_link.stl" />
+        </geometry>
+      </collision>
     </link>
-    <!-- Finger frames share the base axes; meshes use the native CAD placement and the
-         hinges rotate about +X. Zero is closed; the right finger drives, the left mimics. -->
-    <joint name="${prefix}taccap_left_finger_joint" type="revolute">
-      <parent link="${prefix}taccap_base_link"/><child link="${prefix}taccap_left_finger_link"/>
-      <origin xyz="0.0120336718 0.0199500106 0.0484999712" rpy="0 0 0"/>
-      <axis xyz="1 0 0"/>
-      <!-- Effort is the finger motor's maximum output torque; see config/model.json. -->
-      <limit lower="-0.5047492196767601" upper="0" effort="${taccap_finger_effort}" velocity="1"/>
-      <dynamics damping="0.08" friction="0.01"/>
-      <mimic joint="${prefix}taccap_right_finger_joint" multiplier="-1" offset="0"/>
-    </joint>
     <link name="${prefix}taccap_right_finger_link">
       <inertial>
-        <origin xyz="0.020629 0.0066814 0.07491" rpy="0 0 0"/>
-        <mass value="0.36678"/>
-        <inertia ixx="0.00015238" iyy="0.0001547" izz="3.3592e-05" ixy="-2.9549e-07" ixz="-2.4418e-06" iyz="6.6629e-06"/>
+        <origin xyz="0.0140399882 0.003278948264701973 0.04829841241419621" rpy="0 0 0" />
+        <mass value="0.14" />
+        <inertia ixx="0.0003063018651248454" ixy="-1.332880396949135e-06" ixz="-6.566639014047093e-05" iyy="0.0003219105627972025" iyz="-7.90572760751648e-06" izz="3.79806639779513e-05" />
       </inertial>
-      <visual name="${prefix}right_finger_visual">
-        <origin xyz="0 0 0" rpy="${cad_rpy}"/>
-        <geometry><mesh filename="${mesh_root}/grip_right.STL"/></geometry><material name="${prefix}taccap_right_mat"/>
+      <visual name="${prefix}right_link_visual">
+        <origin xyz="1.776356839400251e-18 0 0" rpy="-1.570796326794894 -1.513048197635941 1.570796326794894" />
+        <geometry>
+          <mesh filename="${mesh_root}/right_link.STL" />
+        </geometry>
+        <material name="${prefix}taccap_right_mat" />
       </visual>
-      <collision name="${prefix}right_finger_collision"><origin xyz="0 0 0" rpy="${cad_rpy}"/><geometry><mesh filename="${mesh_root}/grip_right.STL"/></geometry></collision>
+      <collision name="${prefix}right_link_collision">
+        <origin xyz="1.776356839400251e-18 0 0" rpy="-1.570796326794894 -1.513048197635941 1.570796326794894" />
+        <geometry>
+          <mesh filename="${mesh_root}/collision/right_link.stl" />
+        </geometry>
+      </collision>
     </link>
+    <link name="${prefix}taccap_camera_body_link">
+      <inertial>
+        <origin xyz="-0.02305604 9.135000000000001e-05 0.06677412000000001" rpy="0 0 0" />
+        <mass value="0.018" />
+        <inertia ixx="2.08279730304444e-06" ixy="2.468185608919793e-08" ixz="-6.715076777008704e-08" iyy="2.153388567352938e-06" iyz="1.990738215085462e-08" izz="1.83083202960262e-06" />
+      </inertial>
+      <visual name="${prefix}camera_link_visual">
+        <origin xyz="0.01975 -0.0060769 0.034023" rpy="-0 -1.570796326794897 0" />
+        <geometry>
+          <mesh filename="${mesh_root}/camera_link.STL" />
+        </geometry>
+        <material name="${prefix}taccap_base_mat" />
+      </visual>
+      <collision name="${prefix}camera_link_collision">
+        <origin xyz="0.01975 -0.0060769 0.034023" rpy="-0 -1.570796326794897 0" />
+        <geometry>
+          <mesh filename="${mesh_root}/camera_link.STL" />
+        </geometry>
+      </collision>
+    </link>
+    <xacro:if value="${with_mount}">
+      <link name="${prefix}taccap_mount_link">
+        <inertial>
+          <origin xyz="0 0 0.00489788" rpy="0 0 0" />
+          <mass value="0.035" />
+          <inertia ixx="8.044150799999998e-06" ixy="1.145205007058267e-21" ixz="0" iyy="8.044150800000001e-06" iyz="0" izz="1.52699406e-05" />
+        </inertial>
+        <visual name="${prefix}flange_link_visual">
+          <origin xyz="-3.552713678800501e-18 0 -7.105427357601002e-18" rpy="-0 -1.570796326794897 0" />
+          <geometry>
+            <mesh filename="${mesh_root}/flange_link.STL" />
+          </geometry>
+          <material name="${prefix}taccap_cover_mat" />
+        </visual>
+        <collision name="${prefix}flange_link_collision">
+          <origin xyz="-3.552713678800501e-18 0 -7.105427357601002e-18" rpy="-0 -1.570796326794897 0" />
+          <geometry>
+            <mesh filename="${mesh_root}/collision/flange_link.stl" />
+          </geometry>
+        </collision>
+      </link>
+    </xacro:if>
+    <link name="${prefix}taccap_eef_link" />
+    <link name="${prefix}taccap_camera_link" />
+    <link name="${prefix}taccap_camera_optical_link" />
+    <xacro:if value="${with_mount}">
+      <joint name="${prefix}taccap_mount_joint" type="fixed">
+        <parent link="${prefix}taccap_mount_link" />
+        <child link="${prefix}taccap_base_link" />
+        <origin rpy="0 0 0" xyz="0 0 0.012" />
+      </joint>
+    </xacro:if>
+    <joint name="${prefix}taccap_left_finger_joint" type="revolute">
+      <parent link="${prefix}taccap_base_link" />
+      <child link="${prefix}taccap_left_finger_link" />
+      <origin rpy="0 0 0" xyz="0.0120336718 0.0199500106 0.0484999712" />
+      <axis xyz="1 0 0" />
+      <limit effort="1.1" lower="-0.5047492196767601" upper="0" velocity="1" />
+      <dynamics damping="0.08" friction="0.01" />
+      <mimic joint="${prefix}taccap_right_finger_joint" multiplier="-1" offset="0" />
+    </joint>
     <joint name="${prefix}taccap_right_finger_joint" type="revolute">
-      <parent link="${prefix}taccap_base_link"/><child link="${prefix}taccap_right_finger_link"/>
-      <origin xyz="0.0120336718 -0.0199499894 0.0484999712" rpy="0 0 0"/>
-      <axis xyz="1 0 0"/>
-      <limit lower="0" upper="0.5047492196767601" effort="${taccap_finger_effort}" velocity="1"/>
-      <dynamics damping="0.08" friction="0.01"/>
+      <parent link="${prefix}taccap_base_link" />
+      <child link="${prefix}taccap_right_finger_link" />
+      <origin rpy="0 0 0" xyz="0.0120336718 -0.0199499894 0.0484999712" />
+      <axis xyz="1 0 0" />
+      <limit effort="1.1" lower="0" upper="0.5047492196767601" velocity="1" />
+      <dynamics damping="0.08" friction="0.01" />
     </joint>
-    <!-- Massless virtual EEF: centre of the closed fingertips' most distal face (mesh-derived,
-         shared with the master grippers); same axes as taccap_base_link. -->
-    <link name="${prefix}taccap_eef_link"/>
     <joint name="${prefix}taccap_eef_joint" type="fixed">
-      <parent link="${prefix}taccap_base_link"/><child link="${prefix}taccap_eef_link"/>
-      <origin xyz="0.036575 0 0.2009217" rpy="0 0 0"/>
+      <parent link="${prefix}taccap_base_link" />
+      <child link="${prefix}taccap_eef_link" />
+      <origin rpy="0 0 0" xyz="0.036575 0 0.2009217" />
     </joint>
-    <!-- Wrist camera point, from the taccap_base_link origin: 22.75 mm toward -X, 0 in Y,
-         61.25 mm along the tool axis. It lies on the dome-window axis, 19.95 mm behind the window
-         ring. Same axes as taccap_base_link: +Z along the optical (tool) axis, +Y left finger,
-         +X toward the fingers. -->
-    <link name="${prefix}taccap_camera_link"/>
     <joint name="${prefix}taccap_camera_joint" type="fixed">
-      <parent link="${prefix}taccap_base_link"/><child link="${prefix}taccap_camera_link"/>
-      <origin xyz="-0.02275 0 0.06125" rpy="0 0 0"/>
+      <parent link="${prefix}taccap_base_link" />
+      <child link="${prefix}taccap_camera_link" />
+      <origin rpy="0 0 0" xyz="-0.02275 0 0.06125" />
     </joint>
-    <!-- Optical frame (REP-103): +Z optical axis, +X image right, +Y image down toward the fingers. -->
-    <link name="${prefix}taccap_camera_optical_link"/>
     <joint name="${prefix}taccap_camera_optical_joint" type="fixed">
-      <parent link="${prefix}taccap_camera_link"/><child link="${prefix}taccap_camera_optical_link"/>
-      <origin xyz="0 0 0" rpy="0 0 ${-pi/2}"/>
+      <parent link="${prefix}taccap_camera_link" />
+      <child link="${prefix}taccap_camera_optical_link" />
+      <origin rpy="0 0 -1.5707963267948966" xyz="0 0 0" />
+    </joint>
+    <joint name="${prefix}taccap_motor_joint" type="fixed">
+      <parent link="${prefix}taccap_base_link" />
+      <child link="${prefix}taccap_motor_link" />
+      <origin xyz="0 0 0" rpy="0 0 0" />
+    </joint>
+    <joint name="${prefix}taccap_camera_body_joint" type="fixed">
+      <parent link="${prefix}taccap_base_link" />
+      <child link="${prefix}taccap_camera_body_link" />
+      <origin xyz="0 0 0" rpy="0 0 0" />
     </joint>
   </xacro:macro>

File: ros/taccap_description/urdf/taccap_g1_slave_with_mount.urdf (robot description, URDF)
Before this commit: robot taccap_g1_slave_with_mount, 7 links, 6 joints
Links:
- added link taccap_camera_body_link, mass 0.018; collision mesh filename=../meshes/camera_link.STL; visual mesh filename=../meshes/camera_link.STL
- added link taccap_motor_link, mass 0.299; collision mesh filename=../meshes/collision/motor_link.stl; visual mesh filename=../meshes/motor_link.STL
- link taccap_base_link: mass 0.415 -> 0.153; geometry collision mesh filename=../meshes/collision/body_link.stl; visual mesh filename=../meshes/body_link.STL
- link taccap_left_finger_link: mass 0.36678 -> 0.14; geometry collision mesh filename=../meshes/collision/left_link.stl; visual mesh filename=../meshes/left_link.STL
- link taccap_mount_link: mass None -> 0.035; geometry collision mesh filename=../meshes/collision/flange_link.stl; visual mesh filename=../meshes/flange_link.STL
- link taccap_right_finger_link: mass 0.36678 -> 0.14; geometry collision mesh filename=../meshes/collision/right_link.stl; visual mesh filename=../meshes/right_link.STL
Joints:
- added joint taccap_camera_body_joint: type fixed, parent taccap_base_link, child taccap_camera_body_link, origin xyz=0 0 0 rpy=0 0 0
- added joint taccap_motor_joint: type fixed, parent taccap_base_link, child taccap_motor_link, origin xyz=0 0 0 rpy=0 0 0
