Commit message: Streamline the public repository for v0.1.1
- Restructure the READMEs (EN/ZH): key parameters, quick start and links
  to the G1 docs and SDK on the front page; package READMEs cover usage;
  the frame specification lives only in docs/.
- Stop shipping files customers do not use: move the original imported
  URDFs and base mesh to tests/data as regression references, drop the
  unused cover mesh and its USD layer, and remove asset.json.
- base_link.STL is now the canonical body mesh; drop the derivation
  script. Remove internal source details from config/*.json.
- Remove leftovers (cover material name, stale API and comments, unused
  imports), set the maintainer to dylan@xenserobotics.com, and bump the
  version to 0.1.1.

Co-Authored-By: Claude Opus 5.5 <noreply@anthropic.com>

File: ros/taccap_description/urdf/taccap_g1_slave_macro.xacro (robot description, xacro)
@@ -9,5 +9,5 @@
     <material name="${prefix}taccap_left_mat"><color rgba="1 1 1 1"/></material>
     <material name="${prefix}taccap_right_mat"><color rgba="0.60392 0.60392 0.60392 1"/></material>
-    <material name="${prefix}taccap_cover_mat"><color rgba="0.89804 0.91765 0.92941 1"/></material>
+    <material name="${prefix}taccap_mount_mat"><color rgba="0.89804 0.91765 0.92941 1"/></material>
     <!-- taccap_base_link: gripper mounting face (body/Asm_link mating face). +Z along the tool
          axis, +Y toward the left finger, +X toward the off-axis fingers. Meshes keep their native
@@ -21,5 +21,5 @@
           <origin xyz="0 0 0" rpy="${cad_rpy}"/>
           <geometry><mesh filename="${mesh_root}/Asm_link.STL"/></geometry>
-          <material name="${prefix}taccap_cover_mat"/>
+          <material name="${prefix}taccap_mount_mat"/>
         </visual>
         <collision name="${prefix}asm_collision">

File: ros/taccap_master_description/urdf/display_left.urdf.xacro (robot description, xacro)
@@ -1,5 +1,5 @@
 <?xml version="1.0"?>
 <!-- Hand-written standalone wrapper for visualization; NOT generated by
-     scripts/generate_master_models.py. left.urdf.xacro defines a macro rather
+     scripts/generate_master_models.py. taccap_g1_master_left.urdf.xacro defines a macro rather
      than a robot, so robot_state_publisher needs this instantiation. The
      include is relative, so it resolves both in this repository and in the

File: ros/taccap_master_description/urdf/display_right.urdf.xacro (robot description, xacro)
@@ -1,5 +1,5 @@
 <?xml version="1.0"?>
 <!-- Hand-written standalone wrapper for visualization; NOT generated by
-     scripts/generate_master_models.py. right.urdf.xacro defines a macro rather
+     scripts/generate_master_models.py. taccap_g1_master_right.urdf.xacro defines a macro rather
      than a robot, so robot_state_publisher needs this instantiation. The
      include is relative, so it resolves both in this repository and in the
